File: gb_reader.kicad_pcb (KiCad board)
At the start: 2 copper layers, 52 parts, among them J1 Conn_01x32_MountingPin, J2 USB_B_Micro, J3 Conn_01x09, J4 Conn_01x04, J5 Conn_01x32, SW0 SW, SW1 SW, SW2 SW, SW3 SW, U1 STM32F103RFTx, U2 TXB0108DQSR, U3 TXB0108DQSR, U4 TXB0108DQSR, U5 TXB0108DQSR, U6 LM317_3PinPackage, Y1 Crystal_Small

Commit message: pcb layouting
Parts:
- removed C0: 4.7µF, Capacitor_SMD:C_0805_2012Metric
- removed D0: Power LED, LED_SMD:LED_0805_2012Metric
- removed R10: 0, Jumper:SolderJumper-2_P1.3mm_Open_TrianglePad1.0x1.5mm
- removed R11: 10k, Resistor_SMD:R_0603_1608Metric
- removed R12: 440, Resistor_SMD:R_0603_1608Metric
- removed R13: 220, Resistor_SMD:R_0603_1608Metric
- removed R14: 370, Resistor_SMD:R_0603_1608Metric
- removed R9: 1.5k, Resistor_SMD:R_0603_1608Metric
- removed SW0: SW, Button_Switch_THT:SW_TH_Tactile_Omron_B3F-10xx
- removed TP-CLK1, TP-CS1, TP-GND1, TP-RD1, TP-RST1, TP-WR1: , TestPoint:TestPoint_Pad_D2.0mm
- removed TP3V3, TP5V1: TestPoint_Probe, TestPoint:TestPoint_Pad_D2.0mm
- added C11: 100nF, Capacitor_SMD:C_0603_1608Metric, F.Cu at (148.5, 60.0)
- added C12: 100nF, Capacitor_SMD:C_0603_1608Metric, F.Cu at (150.0, 87.5)
- added C13: 100nF, Capacitor_SMD:C_0603_1608Metric, F.Cu at (150.0, 96.5)
- added C14: 100nF, Capacitor_SMD:C_0603_1608Metric, F.Cu at (156.0, 87.5)
- added C15: 100nF, Capacitor_SMD:C_0603_1608Metric, F.Cu at (156.0, 96.5)
- added C16: 100nF, Capacitor_SMD:C_0603_1608Metric, F.Cu at (150.0, 69.5)
- added C17: 100nF, Capacitor_SMD:C_0603_1608Metric, F.Cu at (150.0, 78.5)
- added C18: 100nF, Capacitor_SMD:C_0603_1608Metric, F.Cu at (156.0, 69.5)
- added C19: 100nF, Capacitor_SMD:C_0603_1608Metric, F.Cu at (156.0, 78.5)
- added D1: LED, LED_SMD:LED_0805_2012Metric, F.Cu at (118.5, 81.5)
- added SW4: SW_Push, Button_Switch_SMD:SW_Push_1P1T_NO_CK_KMR2, F.Cu at (144.5, 102.0)
- C10, C8, C9: value 4.7nF -> 100nF
- C2, C3: value 100nF -> 10pF
- C4: value 100nF -> 10µF
- C6, C7: value 10pF -> 100nF
- D2: value LED -> Power LED
- J1: value Conn_01x32_MountingPin -> USB_B_Micro; footprint Connector:DSL_Cartridge_Reader -> Connector_USB:USB_Micro-B_Molex_47346-0001
- J2: value USB_B_Micro -> Conn_01x09; footprint Connector_USB:USB_Micro-B_Molex_47346-0001 -> Connector_PinHeader_2.54mm:PinHeader_1x09_P2.54mm_Horizontal
- J3: value Conn_01x09 -> Conn_01x04; footprint Connector_PinHeader_2.54mm:PinHeader_1x09_P2.54mm_Horizontal -> Connector_PinHeader_2.54mm:PinHeader_1x04_P2.54mm_Horizontal
- J4: value Conn_01x04 -> Conn_01x32; footprint Connector_PinHeader_2.54mm:PinHeader_1x04_P2.54mm_Horizontal -> Connector_PinHeader_2.54mm:PinHeader_1x32_P2.54mm_Vertical
- J5: value Conn_01x32 -> Conn_01x32_MountingPin; footprint Connector_PinHeader_2.54mm:PinHeader_1x32_P2.54mm_Horizontal -> Connector:DSL_Cartridge_Reader
- JP1: value Jumper_NC_Dual -> Jumper_3_Open; footprint Connector_PinHeader_2.54mm:PinHeader_1x03_P2.54mm_Horizontal -> Connector_PinHeader_2.54mm:PinHeader_1x03_P2.54mm_Vertical
- R1: value 1k -> 0; footprint Resistor_SMD:R_0603_1608Metric -> Jumper:SolderJumper-2_P1.3mm_Open_TrianglePad1.0x1.5mm
- R2, R3: value 1k -> 220
- R4: value 1k -> 1.5k
- R5, R6, R7: value 1k -> 100k
- R8: value 440 -> 100k
- SW1, SW2, SW3: value SW -> SW_Push; footprint Button_Switch_THT:SW_TH_Tactile_Omron_B3F-10xx -> Button_Switch_SMD:SW_Push_1P1T_NO_CK_KMR2
- U2: value TXB0108DQSR -> TLV70233_SOT23-5; footprint Package_SON:USON-20_2x4mm_P0.4mm -> Package_TO_SOT_SMD:SOT-23-5
- U3, U4, U5: value TXB0108DQSR -> TXB0108PWR; footprint Package_SON:USON-20_2x4mm_P0.4mm -> Package_SO:TSSOP-20_4.4x6.5mm_P0.65mm
- U6: value LM317_3PinPackage -> TXB0108PWR; footprint Package_TO_SOT_SMD:SOT-223-3_TabPin2 -> Package_SO:TSSOP-20_4.4x6.5mm_P0.65mm
- Y1: value Crystal_Small -> 32kHz
- moved J1 118.5 mm to (135.0, 48.0), turned to 180 degrees
- moved J5 104.7 mm to (198.8, 85.8), turned to 270 degrees
- moved R7 97.0 mm to (143.5, 79.0), turned to 180 degrees
- moved C1 87.4 mm to (140.8, 104.5)
- moved R5 85.9 mm to (143.5, 95.5), turned to 180 degrees
- moved J3 84.2 mm to (116.0, 54.5), turned to 90 degrees
- moved R4 75.4 mm to (130.5, 54.5), turned to 0 degrees
- moved J2 70.6 mm to (89.0, 54.5), turned to 90 degrees
- moved SW1 69.4 mm to (125.0, 77.5), turned to 90 degrees
- moved R6 68.8 mm to (129.5, 95.5), turned to 180 degrees
- moved R8 64.3 mm to (147.0, 87.0), turned to 180 degrees
- moved U2 52.6 mm to (145.5, 61.0), turned to 0 degrees
- moved C5 50.0 mm to (144.5, 82.0), turned to 180 degrees
- moved C6 44.2 mm to (145.5, 91.0), turned to 90 degrees
- moved R3 43.4 mm to (148.5, 56.2), turned to 90 degrees
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Connections:
- C1 pad 1: Pak-Vcc -> /NRST
- C10 pad 1: +3V3 -> +5V
- C2 pad 1: Pak-Vcc -> Net-(C2-Pad1)
- C3 pad 1: Pak-Vcc -> Net-(C3-Pad1)
- C4 pad 1: Pak-Vcc -> GND
- C4 pad 2: GND -> +3V3
- C5 pad 1: Net-(C5-Pad1) -> GND
- C5 pad 2: GND -> +3V3
- C6 pad 1: Net-(C6-Pad1) -> GND
- C6 pad 2: GND -> +3V3
- C7 pad 1: Net-(C7-Pad1) -> GND
- C7 pad 2: GND -> +3V3
- C8 pad 1: +3V3 -> GND
- C8 pad 2: GND -> +3V3
- C9 pad 1: +3V3 -> GND
- C9 pad 2: GND -> +3V3
- D2 pad 1: Net-(D2-Pad1) -> GND
- J1 pad 1: Pak-Vcc -> +5V
- J1 pad 2: CAR_CLK -> USB_DM
- J1 pad 3: CAR_WR -> USB_DP
- J1 pad 4: CAR_RD -> (no net)
- J1 pad 5: CAR_CS -> GND
- J1 pad 6: /Addr0 -> GND
- J2 pad 1: Pak-Vcc -> I2C_SDA
- J2 pad 2: USB_DM -> I2C_SCL
- J2 pad 3: USB_DP -> SPI_MOSI
- J2 pad 4: Net-(J2-Pad4) -> SPI_MISO
- J2 pad 5: GND -> SPI_SCK
- J2 pad 6: GND -> UART4_RX
- J3 pad 1: UART4_TX -> GND
- J3 pad 2: UART4_RX -> SWCLK
- J3 pad 3: SPI_MOSI -> SWDIO
- J3 pad 4: SPI_MISO -> +3V3
- J4 pad 1: GND -> Pak-Vcc
- J4 pad 2: SWCLK -> CAR_CLK
- J4 pad 3: SWDIO -> CAR_WR
- J4 pad 4: +3V3 -> CAR_RD
- JP1 pad 1: Pak-Vcc -> +5V
- R1 pad 1: GND -> /BOOT0
- R1 pad 2: OE-0 -> GND
- R2 pad 1: GND -> /LED
- R2 pad 2: OE-1 -> Net-(D1-Pad2)
- R3 pad 1: GND -> +3V3
- R3 pad 2: OE-2 -> Net-(D2-Pad2)
- R4 pad 1: Net-(R4-Pad1) -> +3V3
- R4 pad 2: GND -> USB_DP
- R5 pad 1: Net-(R5-Pad1) -> GND
- R5 pad 2: GND -> OE-2
- R6 pad 1: Net-(R6-Pad1) -> GND
- R6 pad 2: GND -> OE-3
- R7 pad 2: OE-4 -> OE-0
- R8 pad 1: Pak-Vcc -> GND
- R8 pad 2: Net-(D0-Pad2) -> OE-1
- SW1 pad 1: +3V3 -> GND
- SW1 pad 2: Net-(R4-Pad1) -> /T-A
- SW2 pad 1: +3V3 -> GND
- SW2 pad 2: Net-(R5-Pad1) -> /T-B
- SW3 pad 1: +3V3 -> GND
- SW3 pad 2: Net-(R6-Pad1) -> /T-C
- U1 pad 1: Net-(U1-Pad1) -> +3V3
- U1 pad 10: OE-2 -> /A20
- U1 pad 11: OE-4 -> OE-2
- U1 pad 14: /A3V30 -> /A19
- U1 pad 15: /A3V31 -> /A18
- U1 pad 16: /A3V32 -> /A17
- U1 pad 17: /A3V33 -> /A16
- U1 pad 2: Net-(R5-Pad1) -> ADI
- U1 pad 20: /A3V34 -> /A15
- U1 pad 21: SPI_SCK -> /A14
- U1 pad 22: SPI_MISO -> /A13
- U1 pad 23: SPI_MOSI -> /A12
- U1 pad 24: CAR_RST -> OE-1
- U1 pad 25: /A3V319 -> /A11
- U1 pad 26: /A3V35 -> /A10
- U1 pad 27: /A3V36 -> /A9
- U1 pad 28: /A3V37 -> /A8
- U1 pad 29: /A3V313 -> /A7
- U1 pad 3: Net-(R6-Pad1) -> RST
- U1 pad 30: /A3V314 -> /A6
- U1 pad 33: /A3V315 -> /A5
- U1 pad 34: /A3V316 -> /A4
- U1 pad 35: /A3V317 -> OE-0
- U1 pad 36: /A3V318 -> /A3
- U1 pad 37: /A3V320 -> /A2
- U1 pad 38: /A3V321 -> /A1
- U1 pad 39: /A3V322 -> /A0
- U1 pad 4: Net-(D2-Pad1) -> /A23
- U1 pad 40: /A3V323 -> CS
- U1 pad 41: CAR_WR -> RD
- U1 pad 42: CAR_RD -> WR
- U1 pad 43: CAR_CS -> CLK
- U1 pad 5: Net-(C6-Pad1) -> Net-(C2-Pad1)
- U1 pad 50: ADI -> /T-A
- U1 pad 53: Net-(R4-Pad1) -> /LED
- U1 pad 54: CAR_CLK -> /T-C
- U1 pad 55: /A3V38 -> SPI_SCK
- U1 pad 56: /A3V39 -> SPI_MISO
- U1 pad 57: /A3V310 -> SPI_MOSI
- U1 pad 6: Net-(C7-Pad1) -> Net-(C3-Pad1)
- U1 pad 60: Net-(R10-Pad1) -> /BOOT0
- U1 pad 61: /A3V311 -> /T-B
- U1 pad 62: /A3V312 -> OE-3
- U1 pad 7: Net-(C5-Pad1) -> /NRST
- U1 pad 8: OE-0 -> /A22
- U1 pad 9: OE-1 -> /A21
- U2 pad 1: CAR_CS -> +5V
- U2 pad 2: CAR_RD -> GND
- U2 pad 3: CAR_WR -> +5V
- U2 pad 4: CAR_CLK -> (no net)
- U3 pad 1: /A3V30 -> /A12
- U3 pad 10: /A3V37 -> OE-2
- U3 pad 12: /Addr7 -> /Addr19
- U3 pad 13: /Addr6 -> /Addr18
- U3 pad 14: /Addr5 -> /Addr17
- U3 pad 15: /Addr4 -> /Addr16
- U3 pad 16: /Addr3 -> /Addr15
- U3 pad 17: /Addr2 -> /Addr14
- U3 pad 18: /Addr1 -> /Addr13
- U3 pad 2: /A3V31 -> +3V3
- U3 pad 20: /Addr0 -> /Addr12
- U3 pad 3: /A3V32 -> /A13
- U3 pad 4: /A3V33 -> /A14
- U3 pad 5: +3V3 -> /A15
- U3 pad 6: OE-0 -> /A16
- U3 pad 7: /A3V34 -> /A17
- U3 pad 8: /A3V35 -> /A18
- U3 pad 9: /A3V36 -> /A19
- U4 pad 1: /A3V38 -> /A20
- U4 pad 10: /A3V315 -> OE-3
- U4 pad 12: /Addr15 -> (no net)
- U4 pad 13: /Addr14 -> (no net)
- U4 pad 14: /Addr13 -> CAR_ADI
- U4 pad 15: /Addr12 -> CAR_RST
- U4 pad 16: /Addr11 -> /Addr23
- U4 pad 17: /Addr10 -> /Addr22
- U4 pad 18: /Addr9 -> /Addr21
- U4 pad 2: /A3V39 -> +3V3
- U4 pad 20: /Addr8 -> /Addr20
- U4 pad 3: /A3V310 -> /A21
- U4 pad 4: /A3V311 -> /A22
- U4 pad 5: +3V3 -> /A23
- U4 pad 6: OE-1 -> RST
- U4 pad 7: /A3V312 -> ADI
- U4 pad 8: /A3V313 -> (no net)
- U4 pad 9: /A3V314 -> (no net)
- U5 pad 1: /A3V316 -> CLK
- U5 pad 10: /A3V323 -> OE-0
- U5 pad 12: /Addr23 -> /Addr3
- U5 pad 13: /Addr22 -> /Addr2
- U5 pad 14: /Addr21 -> /Addr1
- U5 pad 15: /Addr20 -> /Addr0
- U5 pad 16: /Addr19 -> CAR_CS
- U5 pad 17: /Addr18 -> CAR_RD
- U5 pad 18: /Addr17 -> CAR_WR
- U5 pad 2: /A3V317 -> +3V3
- U5 pad 20: /Addr16 -> CAR_CLK
- U5 pad 3: /A3V318 -> WR
- U5 pad 4: /A3V319 -> RD
- U5 pad 5: +3V3 -> CS
- U5 pad 6: OE-2 -> /A0
- U5 pad 7: /A3V320 -> /A1
- U5 pad 8: /A3V321 -> /A2
- U5 pad 9: /A3V322 -> /A3
- U6 pad 1: Net-(R13-Pad2) -> /A4
- U6 pad 3: Pak-Vcc -> /A5
- Y1 pad 1: Net-(C6-Pad1) -> Net-(C2-Pad1)
- Y1 pad 2: Net-(C7-Pad1) -> Net-(C3-Pad1)
Routing:
- net +3V3: track 233.2 -> 111.0 mm
- net I2C_SDA: track 0.00 -> 61.1 mm
- net I2C_SCL: track 0.00 -> 59.4 mm
- net Pak-Vcc: track 160.0 -> 102.2 mm
- net SPI_MOSI: track 0.00 -> 57.8 mm
- net SPI_MISO: track 0.00 -> 56.2 mm
- net GND: track 165.5 -> 109.4 mm, vias 4 -> 0
- net SPI_SCK: track 0.00 -> 54.6 mm
- net Net-(R10-Pad1): track 47.3 -> 0.00 mm
- net UART4_RX: track 0.00 -> 45.9 mm
- net OE-3: track 0.00 -> 45.8 mm
- net RST: track 0.00 -> 45.6 mm
- net ADI: track 0.00 -> 45.5 mm
- net /A23: track 0.00 -> 45.4 mm
- net UART4_TX: track 0.00 -> 44.3 mm
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Other:
- rule pad_to_mask_clearance: 0.051 -> 0

Commit message: blo
Parts:
- moved J2 83.3 mm to (143.5, 117.5), turned to 270 degrees
- moved SW2 20.9 mm to (117.8, 69.2)
- moved SW1 8.49 mm to (123.0, 69.2)
- moved SW3 8.27 mm to (112.5, 69.2)
- moved R1 7.39 mm to (117.0, 90.8), turned to 180 degrees
- moved J3 1.75 mm to (117.8, 54.5)
Connections:
- U4 pad 12: (no net) -> GND
- U4 pad 13: (no net) -> GND
- U4 pad 8: (no net) -> GND
- U4 pad 9: (no net) -> GND
Routing:
- net UART4_TX: track 44.3 -> 94.8 mm
- net UART4_RX: track 45.9 -> 94.7 mm
- net /NRST: track 18.7 -> 66.0 mm, vias 0 -> 2
- net +3V3: track 111.0 -> 150.5 mm
- net GND: track 109.4 -> 89.3 mm, vias 0 -> 2
- net /T-B: track 40.5 -> 31.0 mm, vias 0 -> 2
- net /T-A: track 12.2 -> 21.3 mm
- net /T-C: track 26.2 -> 34.7 mm
- net /BOOT0: track 21.6 -> 14.6 mm
- net SPI_SCK: track 54.6 -> 57.7 mm
- net SPI_MISO: track 56.2 -> 58.2 mm
- net SPI_MOSI: track 57.8 -> 59.4 mm
- net I2C_SDA: track 61.1 -> 62.4 mm
- net I2C_SCL: track 59.4 -> 60.7 mm
- net SWCLK: track 35.6 -> 34.9 mm
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- added copper zone on B.Cu, net GND
- added copper zone on F.Cu, net GND
Other:
- board outline added: 142.5 x 87.5 mm

Commit message: Done...löl
Routing:
- net GND: track 89.3 -> 124.5 mm, vias 2 -> 15
- net +3V3: track 150.5 -> 171.6 mm, vias 0 -> 2
- net Pak-Vcc: track 102.2 -> 102.9 mm
Changed lines of the file:
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@@
     (thickness 1.6)
     (drawings 5)
-    (tracks 610)
+    (tracks 670)
     (zones 0)
     (modules 46)
@@
   (layers
     (0 F.Cu signal)
-    (31 B.Cu signal hide)
+    (31 B.Cu signal)
     (32 B.Adhes user)
     (33 F.Adhes user hide)
@@
   (segment (start 145.3 99.2) (end 145.1 99) (width 0.25) (layer F.Cu) (net 1))
   (segment (start 145.3 99.95) (end 145.3 99.2) (width 0.25) (layer F.Cu) (net 1))
+  (via (at 116.25 94) (size 0.8) (drill 0.4) (layers F.Cu B.Cu) (net 1))
+  (via (at 161.25 87.5) (size 0.8) (drill 0.4) (layers F.Cu B.Cu) (net 1))
+  (segment (start 156.925 85.925) (end 157.25 86.25) (width 0.25) (layer F.Cu) (net 1))
+  (segment (start 155.95 85.925) (end 156.925 85.925) (width 0.25) (layer F.Cu) (net 1))
+  (via (at 161 78.25) (size 0.8) (drill 0.4) (layers F.Cu B.Cu) (net 1))
+  (segment (start 155.95 76.925) (end 157.675 76.925) (width 0.25) (layer F.Cu) (net 1))
+  (via (at 161 63.5) (size 0.8) (drill 0.4) (layers F.Cu B.Cu) (net 1))
+  (via (at 140.5 52.5) (size 0.8) (drill 0.4) (layers F.Cu B.Cu) (net 1))
+  (via (at 149 62.75) (size 0.8) (drill 0.4) (layers F.Cu B.Cu) (net 1))
+  (via (at 146.25 78.5) (size 0.8) (drill 0.4) (layers F.Cu B.Cu) (net 1))
+  (segment (start 145.2875 82) (end 144.48749 81.19999) (width 0.25) (layer F.Cu) (net 1))
+  (segment (start 144.48749 81.19999) (end 142.94999 81.19999) (width 0.25) (layer F.Cu) (net 1))
+  (segment (start 142.94999 81.19999) (end 142.715712 81.19999) (width 0.25) (layer F.Cu) (net 1))
+  (segment (start 134 83) (end 134 81.575) (width 0.25) (layer F.Cu) (net 1))
+  (segment (start 141.5 83) (end 134 83) (width 0.25) (layer F.Cu) (net 1))
+  (segment (start 141.75 82.75) (end 141.5 83) (width 0.25) (layer F.Cu) (net 1))
+  (segment (start 142 82.75) (end 141.75 82.75) (width 0.25) (layer F.Cu) (net 1))
+  (segment (start 142.05001 81.19999) (end 142 81.25) (width 0.25) (layer F.Cu) (net 1))
+  (segment (start 142 81.25) (end 142 82.75) (width 0.25) (layer F.Cu) (net 1))
+  (segment (start 142.94999 81.19999) (end 142.05001 81.19999) (width 0.25) (layer F.Cu) (net 1))
+  (via (at 129.5 76) (size 0.8) (drill 0.4) (layers F.Cu B.Cu) (net 1))
+  (segment (start 148.7125 87) (end 149.2125 87.5) (width 0.25) (layer F.Cu) (net 1))
+  (segment (start 147.7875 87) (end 148.7125 87) (width 0.25) (layer F.Cu) (net 1))
+  (via (at 148 88.25) (size 0.8) (drill 0.4) (layers F.Cu B.Cu) (net 1))
+  (segment (start 141 90.5) (end 140.5 91) (width 0.25) (layer F.Cu) (net 1))
+  (via (at 140.5 91) (size 0.8) (drill 0.4) (layers F.Cu B.Cu) (net 1))
+  (segment (start 142.925 90.5) (end 141 90.5) (width 0.25) (layer F.Cu) (net 1))
+  (segment (start 139.934315 91) (end 139 91.934315) (width 0.25) (layer B.Cu) (net 1))
+  (segment (start 140.5 91) (end 139.934315 91) (width 0.25) (layer B.Cu) (net 1))
+  (segment (start 139 91.934315) (end 139 92.5) (width 0.25) (layer B.Cu) (net 1))
+  (via (at 138.5 91) (size 0.8) (drill 0.4) (layers F.Cu B.Cu) (net 1))
+  (segment (start 139 91.5) (end 138.5 91) (width 0.25) (layer F.Cu) (net 1))
+  (segment (start 139 92.925) (end 139 91.5) (width 0.25) (layer F.Cu) (net 1))
+  (via (at 132.25 95) (size 0.8) (drill 0.4) (layers F.Cu B.Cu) (net 1))
+  (via (at 161.25 96.25) (size 0.8) (drill 0.4) (layers F.Cu B.Cu) (net 1))
+  (segment (start 155.95 94.925) (end 157.425 94.925) (width 0.25) (layer F.Cu) (net 1))
+  (segment (start 155.95 102.625) (end 155.95 103.275) (width 0.25) (layer F.Cu) (net 1))
+  (segment (start 132.5375 47.2475) (end 132.09 46.8) (width 0.25) (layer F.Cu) (net 1))
+  (segment (start 132.5375 49.1) (end 132.5375 47.2475) (width 0.25) (layer F.Cu) (net 1))
+  (segment (start 133.7 49.46) (end 133.7 51.2) (width 0.25) (layer F.Cu) (net 1))
+  (segment (start 157.675 77.6125) (end 156.7875 78.5) (width 0.25) (layer F.Cu) (net 1))
+  (segment (start 157.675 76.925) (end 157.675 77.6125) (width 0.25) (layer F.Cu) (net 1))
   (segment (start 135.5 98) (end 135.5 92.925) (width 0.25) (layer F.Cu) (net 2))
   (segment (start 133 100.5) (end 135.5 98) (width 0.25) (layer F.Cu) (net 2))
@@
   (segment (start 150.7875 96.5) (end 151.5 96.5) (width 0.25) (layer F.Cu) (net 4))
   (segment (start 151.5 96.5) (end 151.5 98.5) (width 0.25) (layer F.Cu) (net 4))
-  (segment (start 151.5 89.5) (end 151.5 96.5) (width 0.25) (layer F.Cu) (net 4))
   (segment (start 150.7875 78.5) (end 151.5 78.5) (width 0.25) (layer F.Cu) (net 4))
   (segment (start 151.5 78.5) (end 151.5 71.5) (width 0.25) (layer F.Cu) (net 4))
@@
   (segment (start 136.5 90) (end 139.5 90) (width 0.25) (layer F.Cu) (net 4))
   (segment (start 151.7075 59.2125) (end 153 57.92) (width 0.25) (layer F.Cu) (net 4))
-  (segment (start 151.7075 59.2125) (end 148.5 59.2125) (width 0.25) (layer F.Cu) (net 4))
   (segment (start 146.6 59.475) (end 146.6 60.05) (width 0.25) (layer F.Cu) (net 4))
   (segment (start 146.8625 59.2125) (end 146.6 59.475) (width 0.25) (layer F.Cu) (net 4))
@@
   (segment (start 140.25 43.5) (end 140.25 45.17) (width 0.25) (layer F.Cu) (net 4))
   (segment (start 129.7125 54.5) (end 129.7125 43.5375) (width 0.25) (layer F.Cu) (net 4))
+  (via (at 147 91.5) (size 0.8) (drill 0.4) (layers F.Cu B.Cu) (net 4))
+  (segment (start 145.7125 90.2125) (end 147 91.5) (width 0.25) (layer F.Cu) (net 4))
+  (segment (start 145.5 90.2125) (end 145.7125 90.2125) (width 0.25) (layer F.Cu) (net 4))
+  (segment (start 147 91.5) (end 148.5 90) (width 0.25) (layer B.Cu) (net 4))
+  (segment (start 148.5 90) (end 148.5 89.75) (width 0.25) (layer B.Cu) (net 4))
+  (via (at 151.5 89.75) (size 0.8) (drill 0.4) (layers F.Cu B.Cu) (net 4))
+  (segment (start 148.5 89.75) (end 151.5 89.75) (width 0.25) (layer B.Cu) (net 4))
+  (segment (start 151.5 89.75) (end 151.5 96.5) (width 0.25) (layer F.Cu) (net 4))
+  (segment (start 151.5 89.5) (end 151.5 89.75) (width 0.25) (layer F.Cu) (net 4))
+  (segment (start 151.5 69.5) (end 151.5 68.25) (width 0.25) (layer F.Cu) (net 4))
+  (segment (start 151.5 68.25) (end 154.5 65.25) (width 0.25) (layer F.Cu) (net 4))
+  (segment (start 154.5 62.214998) (end 154.035002 61.75) (width 0.25) (layer F.Cu) (net 4))
+  (segment (start 154.5 65.25) (end 154.5 62.214998) (width 0.25) (layer F.Cu) (net 4))
+  (segment (start 152.550998 61.75) (end 151.25 60.449002) (width 0.25) (layer F.Cu) (net 4))
+  (segment (start 154.035002 61.75) (end 152.550998 61.75) (width 0.25) (layer F.Cu) (net 4))
+  (segment (start 151.25 60.449002) (end 151.25 59.25) (width 0.25) (layer F.Cu) (net 4))
+  (segment (start 151.25 59.25) (end 151.2875 59.2125) (width 0.25) (layer F.Cu) (net 4))
+  (segment (start 151.2875 59.2125) (end 148.5 59.2125) (width 0.25) (layer F.Cu) (net 4))
+  (segment (start 151.7075 59.2125) (end 151.2875 59.2125) (width 0.25) (layer F.Cu) (net 4))
   (segment (start 142.5 59.2125) (end 144.1375 59.2125) (width 0.25) (layer F.Cu) (net 5))
   (segment (start 144.1375 59.2125) (end 144.4 59.475) (width 0.25) (layer F.Cu) (net 5))
@@
   (segment (start 163.38 57.38) (end 155.2125 65.5475) (width 0.25) (layer F.Cu) (net 6))
   (segment (start 163.63 57.13) (end 163.38 57.38) (width 0.25) (layer F.Cu) (net 6))
-  (segment (start 155.2125 62.6725) (end 155.2125 66.7125) (width 0.25) (layer F.Cu) (net 6))
-  (segment (start 153 60.46) (end 155.2125 62.6725) (width 0.25) (layer F.Cu) (net 6))
   (segment (start 155.2125 66.7125) (end 155.2125 68.925) (width 0.25) (layer F.Cu) (net 6))
   (segment (start 155.2125 65.5475) (end 155.2125 66.7125) (width 0.25) (layer F.Cu) (net 6))
+  (segment (start 154.202081 60.46) (end 153 60.46) (width 0.25) (layer F.Cu) (net 6))
+  (segment (start 155.2125 61.470419) (end 154.202081 60.46) (width 0.25) (layer F.Cu) (net 6))
+  (segment (start 155.2125 66.7125) (end 155.2125 61.470419) (width 0.25) (layer F.Cu) (net 6))
   (segment (start 121.2125 83.275) (end 121.2125 83.5) (width 0.25) (layer F.Cu) (net 7))
   (segment (start 119.4375 81.5) (end 121.2125 83.275) (width 0.25) (layer F.Cu) (net 7))
@@
       )
     )
+  )
+  (zone (net 1) (net_name GND) (layer F.Cu) (hatch edge 0.508)
+    (connect_pads (clearance 0.508))
+    (min_thickness 0.254)
+    (fill yes (arc_segments 32) (thermal_gap 0.508) (thermal_bridge_width 0.508))
+    (polygon
+      (pts
+        (xy 85 42.5) (xy 85 130) (xy 227.5 130) (xy 227.5 42.5)
+      )
+    )

Commit message: fixed pcb outline
Other:
- board size 142.5 x 87.5 mm -> 100 x 100 mm
Changed lines of the file:
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@@
   (general
     (thickness 1.6)
-    (drawings 5)
+    (drawings 4)
     (tracks 670)
     (zones 0)
@@
   (layers
     (0 F.Cu signal)
-    (31 B.Cu signal)
+    (31 B.Cu signal hide)
     (32 B.Adhes user)
     (33 F.Adhes user hide)
@@
     )
   )
-  (gr_line (start 85 130) (end 172.5 130) (layer Edge.Cuts) (width 0.1))
-  (gr_line (start 85 42.5) (end 85 130) (layer Edge.Cuts) (width 0.1))
-  (gr_line (start 227.5 42.5) (end 85 42.5) (layer Edge.Cuts) (width 0.1))
-  (gr_line (start 227.5 130) (end 227.5 42.5) (layer Edge.Cuts) (width 0.1))
-  (gr_line (start 172.5 130) (end 227.5 130) (layer Edge.Cuts) (width 0.1))
+  (gr_line (start 208 142.5) (end 208 42.5) (layer Edge.Cuts) (width 0.1))
+  (gr_line (start 108 142.5) (end 208 142.5) (layer Edge.Cuts) (width 0.1))
+  (gr_line (start 108 42.5) (end 208 42.5) (layer Edge.Cuts) (width 0.1))
+  (gr_line (start 108 42.5) (end 108 142.5) (layer Edge.Cuts) (width 0.1))
   (segment (start 150.05 102.625) (end 155.95 102.625) (width 0.25) (layer F.Cu) (net 1))
   (segment (start 150.05 103.275) (end 155.95 103.275) (width 0.25) (layer F.Cu) (net 1))

Commit message: new size
Other:
- board size 100 x 100 mm -> 120 x 87.5 mm
Changed lines of the file:
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@@
     )
   )
-  (gr_line (start 208 142.5) (end 208 42.5) (layer Edge.Cuts) (width 0.1))
-  (gr_line (start 108 142.5) (end 208 142.5) (layer Edge.Cuts) (width 0.1))
-  (gr_line (start 108 42.5) (end 208 42.5) (layer Edge.Cuts) (width 0.1))
-  (gr_line (start 108 42.5) (end 108 142.5) (layer Edge.Cuts) (width 0.1))
+  (gr_line (start 228 42.5) (end 228 130) (layer Edge.Cuts) (width 0.1))
+  (gr_line (start 108 130) (end 228 130) (layer Edge.Cuts) (width 0.1))
+  (gr_line (start 108 42.5) (end 228 42.5) (layer Edge.Cuts) (width 0.1))
+  (gr_line (start 108 42.5) (end 108 130) (layer Edge.Cuts) (width 0.1))
   (segment (start 150.05 102.625) (end 155.95 102.625) (width 0.25) (layer F.Cu) (net 1))
   (segment (start 150.05 103.275) (end 155.95 103.275) (width 0.25) (layer F.Cu) (net 1))
